File: DFO.kicad_pcb (KiCad board)
At the start: 2 copper layers, 18.8 x 18.4 mm, 14 parts, among them U1 Si5351A-B-GT, U2 ATmega328-A, X1 ASE-25MHz

Commit message: update files
Routing:
- net GND: vias 19 -> 20
- net (no net): vias 1 -> 0
Changed lines of the file:
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@@
     (effects (font (size 1 1) (thickness 0.15)))
   )
-  (via (at 108.76 62.95) (size 0.8) (drill 0.4) (layers "F.Cu" "B.Cu") (free) (net 0))
   (segment (start 105.175 77.01) (end 106.759998 77.01) (width 0.45) (layer "F.Cu") (net 1))
   (segment (start 94.41 67.31) (end 94.88 67.31) (width 0.456) (layer "F.Cu") (net 1))
@@
   (via (at 108.65 71.44) (size 0.8) (drill 0.4) (layers "F.Cu" "B.Cu") (free) (net 8))
   (via (at 110.24 73.08) (size 0.8) (drill 0.4) (layers "F.Cu" "B.Cu") (free) (net 8))
+  (via (at 108.76 62.95) (size 0.8) (drill 0.4) (layers "F.Cu" "B.Cu") (free) (net 8))
   (via (at 102.05 65.4) (size 0.8) (drill 0.4) (layers "F.Cu" "B.Cu") (free) (net 8))
   (via (at 99.88 71.52) (size 0.8) (drill 0.4) (layers "F.Cu" "B.Cu") (free) (net 8))
